Commit message: 重新更新文件

File: src/rosrobot_description/urdf/rosrobot.urdf (robot description, URDF)
Before this commit: robot rosrobot, 7 links, 6 joints
Joints:
- joint lh_joint: origin xyz=-0.1391668 0.1725 -0.14 rpy=0 0 0 -> xyz=-0.1391668 0.1925 -0.14 rpy=0 0 0
- joint lq_joint: origin xyz=0.1670723 0.16 -0.0985 rpy=0 0 0 -> xyz=0.1670723 0.14 -0.0985 rpy=0 0 0
- joint rh_joint: origin xyz=-0.1391668 -0.1725 -0.14 rpy=0 0 0 -> xyz=-0.1391668 -0.1925 -0.14 rpy=0 0 0
- joint rq_joint: origin xyz=0.1670723 -0.16 -0.0985 rpy=0 0 0 -> xyz=0.1670723 -0.14 -0.0985 rpy=0 0 0
